File: test.kicad_sch (KiCad schematic)
At the start: 3 parts, among them U1 MSPM0G3507SPTR

Commit message: -
Parts:
- added C3, C5: 470nF, Package_QFP:LQFP-48_7x7mm_P0.5mm, symbol Device:C
- added C4: 10nF, Capacitor_SMD:C_0402_1005Metric_Pad0.74x0.62mm_HandSolder, symbol Device:C
- added R1: 0Ome, symbol Device:R_US
- added R2: 47k, symbol Device:R_US
- added R3: 100k, symbol Device:R_US
Connections:
- net +3V3: now also R2.1
- net Earth: now also C4.2, C5.2, R1.2, R3.1; no longer U1.7 (VSS)
- net VREF-: now reaches U1.39 (PA21)
- net VREF-: now also C3.2, R1.1
- net NRTS: now reaches U1.4 (NRST)
- net NRTS: now also C4.1, R2.2
- net VREF+: now reaches U1.43 (PA23)
- net VREF+: now also C3.1
- net ROSC ±0.1% ±25ppm: now reaches U1.8 (PA2)
- net ROSC ±0.1% ±25ppm: now also R3.2
- new net: C5.1, U1.7 (VSS)
